File: pcb/nokia.kicad_pcb (KiCad board)
At the start: 4 copper layers, 42.1 x 108 mm, 88 parts, among them J1 Conn_01x07, J2 USB_B_Micro, J20 Conn_01x04_Pin, J3 SM03B-SRSS-TB, J6 SM03B-SRSS-TB, M1 Vibration, Q1 BC847, SW1 SW_Push, U1 W25Q128JVS, U4 NCP1117-3.3_SOT223, U5 RP2350_80QFN, Y1 ABM8-272-T3, Y2 RV-3028-C7_32.768kHz_1ppm_TA_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

Commit message: pcb v0.3
Parts:
- removed C22: 100n, Capacitor_SMD:C_0402_1005Metric
- removed J6: SM03B-SRSS-TB, Connector_JST:JST_SH_SM03B-SRSS-TB_1x03-1MP_P1.00mm_Horizontal
- removed R17: 90, Resistor_SMD:R_0402_1005Metric
- added C25: 10u, Capacitor_SMD:C_0805_2012Metric, B.Cu at (50.0, 49.8)
- added C26: 100nF, Capacitor_SMD:C_0805_2012Metric, B.Cu at (26.6, 37.2)
- added C27: 22uF, Capacitor_SMD:C_0805_2012Metric, B.Cu at (26.6, 35.2)
- added C28: 22uF, Capacitor_SMD:C_0805_2012Metric, B.Cu at (26.6, 33.1)
- added C29: 100nF, Capacitor_SMD:C_0805_2012Metric, B.Cu at (25.8, 46.5)
- added C30: 22uF, Capacitor_SMD:C_0805_2012Metric, B.Cu at (27.8, 46.5)
- added C33: 47uF, Capacitor_SMD:C_0805_2012Metric, B.Cu at (53.8, 24.8)
- added C34: 1uF, Capacitor_SMD:C_0805_2012Metric, B.Cu at (26.8, 28.9)
- added C35: 22uF, Capacitor_SMD:C_0805_2012Metric, B.Cu at (29.8, 46.5)
- added D10: BAS16J, Diode_SMD:D_SOD-323F, B.Cu at (46.9, 27.0)
- added D12: SS34, Diode_SMD:D_SMA, B.Cu at (27.8, 51.8)
- added D2: LED, LED_SMD:LED_REVERSE, B.Cu at (27.5, 74.3)
- added D3: LED, LED_SMD:LED_REVERSE, B.Cu at (37.9, 74.3)
- added D4: LED, LED_SMD:LED_REVERSE, B.Cu at (47.1, 74.3)
- added D5: LED, LED_SMD:LED_REVERSE, B.Cu at (34.8, 113.9)
- added D6: LED, LED_SMD:LED_REVERSE, B.Cu at (50.2, 113.3)
- added D7: LED, LED_SMD:LED_REVERSE, B.Cu at (35.0, 100.0)
- added D8: LED, LED_SMD:LED_REVERSE, B.Cu at (50.2, 99.8)
- added D9: LED, LED_SMD:LED_REVERSE, B.Cu at (57.5, 74.4)
- added F1: Polyfuse, Fuse:Fuse_Bourns_MF-SM_7.98x5.44mm, B.Cu at (59.7, 38.0)
- added J5: USB_B_Micro, Connector_USB:USB_Micro-B_Molex_47346-0001, B.Cu at (38.2, 123.8)
- added JP2: Jumper_2_Open, Jumper:SolderJumper-2_P1.3mm_Open_RoundedPad1.0x1.5mm, B.Cu at (36.8, 38.0)
- added L2: 4.7uH, Inductor_SMD:L_Neosid_MicroCoil_Ms36-L, B.Cu at (34.4, 30.1)
- added Q2: BC847, Package_TO_SOT_SMD:SOT-23, B.Cu at (31.5, 73.6)
- added Q4: BSS138, Package_TO_SOT_SMD:SOT-23, B.Cu at (42.5, 22.4)
- added Q5: BC847, Package_TO_SOT_SMD:SOT-23, B.Cu at (53.1, 113.7)
- added Q6: BSS138, Package_TO_SOT_SMD:SOT-23, B.Cu at (56.3, 29.2)
- added Q7: BC847, Package_TO_SOT_SMD:SOT-23, B.Cu at (47.1, 99.9)
- added Q9: BC847, Package_TO_SOT_SMD:SOT-23, B.Cu at (53.2, 73.5)
- added R11: 220, Resistor_SMD:R_0402_1005Metric, B.Cu at (36.7, 98.3)
- added R12: 220, Resistor_SMD:R_0402_1005Metric, B.Cu at (48.1, 97.5)
- added R13: 220, Resistor_SMD:R_0402_1005Metric, B.Cu at (56.7, 72.5)
- added R14: 1K, Resistor_SMD:R_0402_1005Metric, B.Cu at (45.2, 21.8)
- added R15: 100k, Resistor_SMD:R_0402_1005Metric, B.Cu at (59.4, 33.1)
- added R16: 1K, Resistor_SMD:R_0402_1005Metric, B.Cu at (59.8, 29.9)
- added R18: 100, Resistor_SMD:R_0402_1005Metric, B.Cu at (53.3, 27.4)
- added R19: 1K, Resistor_SMD:R_0402_1005Metric, B.Cu at (55.1, 31.8)
- added R20: 10k, Resistor_SMD:R_0402_1005Metric, B.Cu at (55.1, 33.0)
- added R21: 200k, Resistor_SMD:R_0402_1005Metric, B.Cu at (53.3, 26.4)
- added R22: 1K, Resistor_SMD:R_0402_1005Metric, B.Cu at (30.4, 23.9)
- added R4: 220, Resistor_SMD:R_0402_1005Metric, B.Cu at (28.9, 72.7)
- added R41: 1K, Resistor_SMD:R_0402_1005Metric, B.Cu at (27.2, 44.2)
- added R5: 220, Resistor_SMD:R_0402_1005Metric, B.Cu at (36.5, 72.7)
- added SW2: SW_Push, Button_Switch_SMD:SW_SPST_PTS810, B.Cu at (56.9, 35.9)
- added TP1: TestPoint, TestPoint:TestPoint_THTPad_D1.5mm_Drill0.7mm, F.Cu at (24.6, 54.4)
- added TP2: TestPoint, TestPoint:TestPoint_THTPad_D1.5mm_Drill0.7mm, F.Cu at (24.4, 51.0)
- added U2: NCP1117-3.3_SOT223, Package_TO_SOT_SMD:SOT-223-3_TabPin2, B.Cu at (57.5, 50.4)
- added U3: TP5400, Package_SO:SOIC-8_3.9x4.9mm_P1.27mm, B.Cu at (27.5, 40.9)
- added U6: 74LVC1G14, Package_TO_SOT_SMD:SOT-23-5_HandSoldering, B.Cu at (40.6, 33.0)
- added U7: 74LVC1G17, Package_TO_SOT_SMD:SOT-23-5_HandSoldering, B.Cu at (42.9, 26.1)
- added U8: 74LVC1G175, Package_TO_SOT_SMD:TSOT-23-6_HandSoldering, B.Cu at (48.9, 22.9)
- C1: value 10u -> 22uF
- C23: value 100m, 5V5 -> 10u; footprint CoreElectronics_Components:Kemet_FC_10.5X5.5 -> Capacitor_SMD:C_0805_2012Metric
- C5: value 10u -> 100n; footprint Capacitor_SMD:C_0805_2012Metric -> Capacitor_SMD:C_0402_1005Metric
- J2: value USB_B_Micro -> Conn_02x04_Counter_Clockwise; footprint Connector_USB:USB_Micro-B_Amphenol_10103594-0001LF_Horizontal -> Connector_PinHeader_2.54mm:PinHeader_2x04_P2.54mm_Vertical_SMD
- J3: value SM03B-SRSS-TB -> Conn_01x02_Pin; footprint Connector_JST:JST_SH_SM03B-SRSS-TB_1x03-1MP_P1.00mm_Horizontal -> Connector_PinHeader_1.00mm:PinHeader_1x02_P1.00mm_Vertical_SMD_Pin1Left; moved to F.Cu
- R1: value DNF -> 10k
- R10: value 0 -> 220
- R6: value 3k -> 220
- R9: value DNF -> 220
- U4: value NCP1117-3.3_SOT223 -> SIL2308; footprint Package_TO_SOT_SMD:SOT-223-3_TabPin2 -> Package_TO_SOT_SMD:SOT-23-6
- moved J3 95.9 mm to (42.6, 28.0), turned to 0 degrees
- moved J2 90.3 mm to (48.3, 33.9), turned to 90 degrees
- moved C23 61.6 mm to (50.0, 46.4), turned to -90 degrees
- moved C1 55.2 mm to (30.9, 37.2), turned to 180 degrees
- moved R9 53.5 mm to (36.9, 115.2), turned to 180 degrees
- moved R10 51.9 mm to (52.4, 111.3), turned to 180 degrees
- moved R6 50.2 mm to (48.5, 72.7), turned to 180 degrees
- moved U4 44.6 mm to (57.7, 43.2)
- moved C5 11.9 mm to (39.5, 95.5), turned to -90 degrees
- moved Q1 6.63 mm to (56.9, 95.0)
- moved R47 3.27 mm to (56.4, 110.6), turned to -90 degrees
- moved D1 2.36 mm to (55.3, 97.8), turned to 90 degrees
- moved M1 2.33 mm to (55.5, 111.3)
- moved R37 1.60 mm to (44.0, 96.5)
- moved R8 1.60 mm to (55.7, 58.2)
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Connections:
- C1 pad 2: GND -> -BATT
- C10 pad 2: GND -> -BATT
- C11 pad 2: GND -> -BATT
- C12 pad 2: GND -> -BATT
- C13 pad 2: GND -> -BATT
- C14 pad 2: GND -> -BATT
- C15 pad 2: GND -> -BATT
- C16 pad 2: GND -> -BATT
- C17 pad 2: GND -> -BATT
- C18 pad 2: GND -> -BATT
- C19 pad 2: GND -> -BATT
- C2 pad 2: GND -> -BATT
- C20 pad 2: GND -> -BATT
- C21 pad 2: GND -> -BATT
- C23 pad 1: Net-(Y2-VBACKUP) -> Net-(U2-VI)
- C23 pad 2: GND -> -BATT
- C24 pad 2: GND -> -BATT
- C3 pad 2: GND -> -BATT
- C4 pad 2: GND -> -BATT
- C5 pad 1: +3V3 -> Net-(Y2-VBACKUP)
- C5 pad 2: GND -> -BATT
- C6 pad 2: GND -> -BATT
- C7 pad 2: GND -> -BATT
- C79 pad 1: GND -> -BATT
- C8 pad 2: GND -> -BATT
- C9 pad 2: GND -> -BATT
- J1 pad 6: GND -> -BATT
- J2 pad 1: VBUS -> -BATT
- J2 pad 2: /USB_D- -> /SWCLK
- J2 pad 3: /USB_D+ -> -BATT
- J2 pad 4: unconnected-(J2-ID-Pad4) -> /SWD
- J2 pad 5: GND -> /GPIO0
- J2 pad 6: GND -> -BATT
- J20 pad 1: +3V3 -> +BATT
- J20 pad 4: GND -> -BATT
- J3 pad 1: /GPIO1 -> /GPIO34
- J3 pad 2: GND -> -BATT
- KP#1 pad 1: GND -> -BATT
- KP*1 pad 1: GND -> -BATT
- KP0 pad 1: GND -> -BATT
- KP1 pad 1: GND -> -BATT
- KP2 pad 1: GND -> -BATT
- KP3 pad 1: GND -> -BATT
- KP4 pad 1: GND -> -BATT
- KP5 pad 1: GND -> -BATT
- KP6 pad 1: GND -> -BATT
- KP7 pad 1: GND -> -BATT
- KP8 pad 1: GND -> -BATT
- KP9 pad 1: GND -> -BATT
- KPC1 pad 1: GND -> -BATT
- KPDOWN1 pad 1: GND -> -BATT
- KPSELECT1 pad 1: GND -> -BATT
- KPUP1 pad 1: GND -> -BATT
- LS2 pad 2: GND -> -BATT
- Q1 pad 2: GND -> -BATT
- R1 pad 1: +3V3 -> /QSPI_SS
- R1 pad 2: /FLASH_SS -> Net-(R1-Pad2)
- R10 pad 1: /QSPI_SS -> Net-(Q5-C)
- R10 pad 2: /FLASH_SS -> Net-(D6-K)
- R39 pad 2: GND -> -BATT
- R6 pad 1: +3V3 -> Net-(Q9-C)
- R6 pad 2: /GPIO28 -> Net-(D4-K)
- R9 pad 1: /GPIO0 -> Net-(Q5-C)
- R9 pad 2: /FLASH_SS -> Net-(D5-K)
- SW1 pad 1: GND -> -BATT
- SW1 pad 2: /GPIO28 -> /Btn
- U1 pad 1: /FLASH_SS -> /QSPI_SS
- U1 pad 4: GND -> -BATT
- U4 pad 1: GND -> Net-(R16-Pad2)
- U4 pad 2: +3V3 -> Net-(F1-Pad1)
- U4 pad 3: VBUS -> Net-(R15-Pad1)
- U5 pad 22: /GPIO22 -> unconnected-(U5-GPIO22-Pad22)
- U5 pad 23: /GPIO23 -> unconnected-(U5-GPIO23-Pad23)
- U5 pad 25: /GPIO24 -> unconnected-(U5-GPIO24-Pad25)
- U5 pad 26: /GPIO25 -> unconnected-(U5-GPIO25-Pad26)
- U5 pad 27: /GPIO26 -> unconnected-(U5-GPIO26-Pad27)
- U5 pad 28: /GPIO27 -> unconnected-(U5-GPIO27-Pad28)
- U5 pad 36: /GPIO28 -> /Btn
- U5 pad 37: /GPIO29 -> unconnected-(U5-GPIO29-Pad37)
- U5 pad 38: /GPIO30 -> unconnected-(U5-GPIO30-Pad38)
- U5 pad 39: /GPIO31 -> unconnected-(U5-GPIO31-Pad39)
- U5 pad 40: /GPIO32 -> unconnected-(U5-GPIO32-Pad40)
- U5 pad 44: /GPIO35 -> unconnected-(U5-GPIO35-Pad44)
- U5 pad 49: /GPIO40_ADC0 -> unconnected-(U5-GPIO40_ADC0-Pad49)
- U5 pad 52: /GPIO41_ADC1 -> unconnected-(U5-GPIO41_ADC1-Pad52)
- U5 pad 54: /ALARMB -> unconnected-(U5-GPIO43_ADC3-Pad54)
- U5 pad 55: /SDA0 -> unconnected-(U5-GPIO44_ADC4-Pad55)
- U5 pad 56: /SCL0 -> unconnected-(U5-GPIO45_ADC5-Pad56)
- U5 pad 62: GND -> -BATT
- U5 pad 80: /GPIO3 -> unconnected-(U5-GPIO3-Pad80)
- U5 pad 81: GND -> -BATT
- Y1 pad 2: GND -> -BATT
- Y1 pad 4: GND -> -BATT
- Y2 pad 1: /CLK -> unconnected-(Y2-CLKOUT-Pad1)
- Y2 pad 5: GND -> -BATT
Routing:
- net -BATT: track 0.00 -> 292.2 mm, vias 0 -> 84
- net /GPIO15: track 0.00 -> 101.8 mm, vias 0 -> 3
- net +5V: track 0.00 -> 88.9 mm, vias 0 -> 10
- net /Btn: track 0.00 -> 86.6 mm, vias 0 -> 5
- net VBUS: track 39.8 -> 123.4 mm, vias 2 -> 3
- net GND: track 69.8 -> 0.00 mm, vias 86 -> 0
- net /GPIO1: track 84.8 -> 30.3 mm
- net /GPIO0: track 94.7 -> 50.5 mm, vias 3 -> 2
- net /GPIO28: track 43.1 -> 0.00 mm
- net /SWD: track 83.2 -> 41.8 mm, vias 2 -> 3
- net /SWCLK: track 83.0 -> 46.8 mm
- net Net-(R1-Pad2): track 0.00 -> 32.9 mm, vias 0 -> 2
- net +BATT: track 0.00 -> 31.2 mm, vias 0 -> 2
- net Net-(D12-A): track 0.00 -> 28.4 mm, vias 0 -> 2
- net /GPIO10: track 56.3 -> 83.1 mm, vias 2 -> 3
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- added copper zone on B.Cu, net -BATT
- added copper zone on F.Cu, net -BATT
- added copper zone on In2.Cu, net -BATT
- removed copper zone on B.Cu, net GND
- removed copper zone on F.Cu, net GND
- removed copper zone on In2.Cu, net GND
Other:
- outline, holes or cut-outs redrawn
