File: pcb/nokia.kicad_sch (KiCad schematic)
At the start: 122 parts, among them J1 Conn_01x07, J2 USB_B_Micro, J20 Conn_01x04_Pin, J3 SM03B-SRSS-TB, J5 Conn_01x03_Pin, J6 SM03B-SRSS-TB, J7 Conn_01x03_Pin, M1 Vibration, Q1 BC847, SW1 SW_Push, U1 W25Q128JVS, U4 NCP1117-3.3_SOT223, U5 RP2350_80QFN, Y1 ABM8-272-T3, Y2 RV-3028-C7_32.768kHz_1ppm_TA_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

Commit message: pcb v0.3
Parts:
- removed C23: 100m, 5V5, CoreElectronics_Components:Kemet_FC_10.5X5.5, symbol PiicoDev-Real-Time-Clock-RV3028-rescue:CP1-Device
- removed C5: 10u, Capacitor_SMD:C_0805_2012Metric, symbol Device:C
- removed D2, D3, D4, D5, D6, D7, D8, D9: LED_ARGB, LED_SMD:RGBLED-reverse, symbol Device:LED_ARGB
- removed J2: USB_B_Micro, Connector_USB:USB_Micro-B_Amphenol_10103594-0001LF_Horizontal, symbol Connector:USB_B_Micro
- removed J3, J6: SM03B-SRSS-TB, Connector_JST:JST_SH_SM03B-SRSS-TB_1x03-1MP_P1.00mm_Horizontal, symbol Connector_Generic_MountingPin:Conn_01x03_MountingPin
- removed J5, J7: Conn_01x03_Pin, Connector_PinHeader_2.54mm:PinHeader_1x03_P2.54mm_Vertical, symbol Connector:Conn_01x03_Pin
- removed R10: 0, Resistor_SMD:R_0402_1005Metric, symbol Device:R
- removed R11, R12, R14, R15, R16, R17, R19, R20, R22, R23, R25, R26, R28, R29, R31, R32: 90, Resistor_SMD:R_0402_1005Metric, symbol Device:R
- removed R13, R18, R21, R24, R27, R30, R4, R5: 140, Resistor_SMD:R_0402_1005Metric, symbol Device:R
- removed R6: 3k, Resistor_SMD:R_0402_1005Metric, symbol Device:R
- removed R9: DNF, Resistor_SMD:R_0402_1005Metric, symbol Device:R
- removed U4: NCP1117-3.3_SOT223, Package_TO_SOT_SMD:SOT-223-3_TabPin2, symbol Regulator_Linear:NCP1117-3.3_SOT223
- added C23, C25: 10u, Capacitor_SMD:C_0805_2012Metric, symbol Device:C
- added C26, C29: 100nF, Capacitor_SMD:C_0805_2012Metric, symbol Device:C
- added C27, C28, C30, C35: 22uF, Capacitor_SMD:C_0805_2012Metric, symbol Device:C
- added D12: SS34, Diode_SMD:D_SMC, symbol Device:D_Schottky
- added J2: Conn_02x04_Counter_Clockwise, Connector_PinHeader_2.54mm:PinHeader_2x04_P2.54mm_Vertical_SMD, symbol Connector_Generic:Conn_02x04_Counter_Clockwise
- added J3: Conn_01x02_Pin, Connector_PinHeader_1.00mm:PinHeader_1x02_P1.00mm_Vertical_SMD_Pin1Left, symbol Connector:Conn_01x02_Pin
- added J4: USB_C_Receptacle_USB2.0_14P, Connector_USB:USB_C_Receptacle_GCT_USB4105-xx-A_16P_TopMnt_Horizontal, symbol Connector:USB_C_Receptacle_USB2.0_14P
- added J5: Conn_01x04, Connector_PinHeader_2.54mm:PinHeader_1x04_P2.54mm_Vertical_SMD_Pin1Right, symbol Connector_Generic:Conn_01x05
- added JP1: Jumper_2_Open, Jumper:SolderJumper-2_P1.3mm_Open_RoundedPad1.0x1.5mm, symbol Jumper:Jumper_2_Open
- added L2: 4.7uH, symbol Device:L
- added R33, R40: 5.1k, Resistor_SMD:R_0402_1005Metric, symbol Device:R
- added R41: 1K, Resistor_SMD:R_0402_1005Metric, symbol Device:R
- added SW2: SW_Push, Button_Switch_SMD:SW_SPST_PTS810, symbol Switch:SW_Push
- added TP2: TestPoint, TestPoint:TestPoint_THTPad_D1.5mm_Drill0.7mm, symbol Connector:TestPoint
- added U2: NCP1117-3.3_SOT223, Package_TO_SOT_SMD:SOT-223-3_TabPin2, symbol Regulator_Linear:NCP1117-3.3_SOT223
- added U3: TP5400, Package_SO:SOIC-8_3.9x4.9mm_P1.27mm, symbol Interface_CAN_LIN:SN65HVD255D
- C1: value 10u -> 22uF
- R1: value DNF -> 10k
- TP1: footprint PiicoDev Real Time Clock RV3028:PinHeader_1x01_P2.54mm_Vertical -> TestPoint:TestPoint_THTPad_D1.5mm_Drill0.7mm
Connections:
- net +3V3: now also C25.1, U2.2 (VO); no longer J20.1 (Pin_1), R1.1
- net GPIO0: now also J2.5 (Pin_5)
- net GPIO1: now also J2.7 (Pin_7)
- net GPIO21: now also J5.4 (Pin_4), J5.5 (Pin_5)
- net GPIO34: now also J3.1 (Pin_1), J5.3 (Pin_3)
- net QSPI_SS: now also R1.1, U1.1 (~{CS})
- net SWCLK: now also J2.2 (Pin_2)
- net SWD: now also J2.4 (Pin_4)
- net USB_D+: now also J4.A7 (D-), J4.B7 (D-)
- net USB_D-: now also J4.A6 (D+), J4.B6 (D+)
- net VBUS: now also J4.A4 (VBUS), J4.A9 (VBUS), J4.B4 (VBUS), J4.B9 (VBUS), JP1.1 (A), U3.5 (VCC)
- net at C22.1, Y2.6 (VBACKUP): no longer TP1.1
- net ALARMB: no longer names the net of U5.54 (GPIO43_ADC3)
- net CLK: no longer names the net of Y2.1 (CLKOUT)
- net FLASH_SS: no longer names the net of R1.2
- net FLASH_SS: now also SW2.2; no longer U1.1 (~{CS})
- net GND renamed -BATT
- net -BATT: now also C23.2, C25.2, C26.2, C27.2, C28.2, C29.1, C30.1, C35.1, J2.1 (Pin_1), J2.3 (Pin_3), J2.6 (Pin_6), J3.2 (Pin_2), J4.A1 (GND), J4.A12 (GND), J4.B1 (GND), J4.B12 (GND), J4.S1 (SHIELD), J5.1 (Pin_1), J5.2 (Pin_2), R33.1, R40.1, R41.1, SW2.1, U2.1 (GND), U3.7 (GND)
- net GPIO15: no longer names the net of U5.14 (GPIO15)
- net GPIO22: no longer names the net of U5.22 (GPIO22)
- net GPIO23: no longer names the net of U5.23 (GPIO23)
- net GPIO24: no longer names the net of U5.25 (GPIO24)
- net GPIO25: no longer names the net of U5.26 (GPIO25)
- net GPIO26: no longer names the net of U5.27 (GPIO26)
- net GPIO27: no longer names the net of U5.28 (GPIO27)
- net GPIO29: no longer names the net of U5.37 (GPIO29)
- net GPIO3: no longer names the net of U5.80 (GPIO3)
- net GPIO30: no longer names the net of U5.38 (GPIO30)
- net GPIO31: no longer names the net of U5.39 (GPIO31)
- net GPIO32: no longer names the net of U5.40 (GPIO32)
- net GPIO35: no longer names the net of U5.44 (GPIO35)
- net GPIO40_ADC0: no longer names the net of U5.49 (GPIO40_ADC0)
- net GPIO41_ADC1: no longer names the net of U5.52 (GPIO41_ADC1)
- net SCL0: no longer names the net of U5.56 (GPIO45_ADC5)
- net SDA0: no longer names the net of U5.55 (GPIO44_ADC4)
- new net: TP2.1, U3.4 (STDBY)
- new net: D12.2 (A), L2.1, U3.8 (LX)
- new net: R41.2, U3.3 (PROG)
- new net: J4.A5 (CC1), R33.2
- new net: J4.B5 (CC2), R40.2
- new net: TP1.1, U3.2 (CHRG)
- new net +5V: C23.1, C29.2, C30.2, C35.2, D12.1 (K), J2.8 (Pin_8), JP1.2 (B), U2.3 (VI), U3.1 (VOUT)
- new net +BATT: C26.1, C27.1, C28.1, J20.1 (Pin_1), L2.2, U3.6 (BAT)
- no-connect marks 4 -> 23
Other:
- note added: "Charging"
- note removed: "Clear jumper to remove I2C pullup"
- note removed: "JST Debug Connector"
- note removed: "UART Connector"
- moved on the sheet: C22, C24, C3, C4, C79, J20, KP#1, KP*1, KP0, KP1, KP2, KP3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
