File: pcb/nokia.kicad_sch (KiCad schematic)
At the start: 122 parts, among them J1 Conn_01x07, J2 USB_B_Micro, J20 Conn_01x04_Pin, J3 SM03B-SRSS-TB, J5 Conn_01x03_Pin, J6 SM03B-SRSS-TB, J7 Conn_01x03_Pin, M1 Vibration, Q1 BC847, SW1 SW_Push, U1 W25Q128JVS, U4 NCP1117-3.3_SOT223, U5 RP2350_80QFN, Y1 ABM8-272-T3, Y2 RV-3028-C7_32.768kHz_1ppm_TA_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

Commit message: pcb v0.3
Parts:
- removed C22: 100n, Capacitor_SMD:C_0402_1005Metric, symbol Device:C
- removed C23: 100m, 5V5, CoreElectronics_Components:Kemet_FC_10.5X5.5, symbol PiicoDev-Real-Time-Clock-RV3028-rescue:CP1-Device
- removed D2, D3, D4, D5, D6, D7, D8, D9: LED_ARGB, LED_SMD:RGBLED-reverse, symbol Device:LED_ARGB
- removed J2: USB_B_Micro, Connector_USB:USB_Micro-B_Amphenol_10103594-0001LF_Horizontal, symbol Connector:USB_B_Micro
- removed J3, J6: SM03B-SRSS-TB, Connector_JST:JST_SH_SM03B-SRSS-TB_1x03-1MP_P1.00mm_Horizontal, symbol Connector_Generic_MountingPin:Conn_01x03_MountingPin
- removed J5, J7: Conn_01x03_Pin, Connector_PinHeader_2.54mm:PinHeader_1x03_P2.54mm_Vertical, symbol Connector:Conn_01x03_Pin
- removed R17, R23, R25, R26, R28, R29, R31, R32: 90, Resistor_SMD:R_0402_1005Metric, symbol Device:R
- removed R24, R27, R30: 140, Resistor_SMD:R_0402_1005Metric, symbol Device:R
- removed U4: NCP1117-3.3_SOT223, Package_TO_SOT_SMD:SOT-223-3_TabPin2, symbol Regulator_Linear:NCP1117-3.3_SOT223
- added C23, C25: 10u, Capacitor_SMD:C_0805_2012Metric, symbol Device:C
- added C26, C29: 100nF, Capacitor_SMD:C_0805_2012Metric, symbol Device:C
- added C27, C28, C30, C35: 22uF, Capacitor_SMD:C_0805_2012Metric, symbol Device:C
- added C31: 100m, 5V5, CoreElectronics_Components:Kemet_FC_10.5X5.5, symbol PiicoDev-Real-Time-Clock-RV3028-rescue:CP1-Device
- added C33: 47uF, Capacitor_SMD:C_0805_2012Metric, symbol Device:C
- added C34: 1uF, Capacitor_SMD:C_0805_2012Metric, symbol Device:C
- added D10: BAS16J, Diode_SMD:D_SOD-323F, symbol Device:D
- added D12: SS34, Diode_SMD:D_SMA, symbol Device:D_Schottky
- added D2, D3, D4, D5, D6, D7, D8, D9: LED, LED_REVERSE, symbol Device:LED
- added F1: Polyfuse, Fuse:Fuse_Bourns_MF-SM_7.98x5.44mm, symbol Device:Polyfuse
- added J2: Conn_02x04_Counter_Clockwise, Connector_PinHeader_2.54mm:PinHeader_2x04_P2.54mm_Vertical_SMD, symbol Connector_Generic:Conn_02x04_Counter_Clockwise
- added J3: Conn_01x02_Pin, Connector_PinHeader_1.00mm:PinHeader_1x02_P1.00mm_Vertical_SMD_Pin1Left, symbol Connector:Conn_01x02_Pin
- added J5: USB_B_Micro, Connector_USB:USB_Micro-B_Molex_47346-0001, symbol Connector:USB_B_Micro
- added JP2: Jumper_2_Open, Jumper:SolderJumper-2_P1.3mm_Open_RoundedPad1.0x1.5mm, symbol Jumper:Jumper_2_Open
- added L2: 4.7uH, Inductor_SMD:L_Neosid_MicroCoil_Ms36-L, symbol Device:L
- added Q2, Q5, Q7, Q9: BC847, Package_TO_SOT_SMD:SOT-23, symbol Transistor_BJT:BC847
- added Q4, Q6: BSS138, Package_TO_SOT_SMD:SOT-23, symbol Transistor_FET:BSS138
- added R41: 1K, Resistor_SMD:R_0402_1005Metric, symbol Device:R
- added SW2: SW_Push, Button_Switch_SMD:SW_SPST_PTS810, symbol Switch:SW_Push
- added TP2: TestPoint, TestPoint:TestPoint_THTPad_D1.5mm_Drill0.7mm, symbol Connector:TestPoint
- added TP3: TestPoint, PiicoDev Real Time Clock RV3028:PinHeader_1x01_P2.54mm_Vertical, symbol Connector:TestPoint
- added U2: NCP1117-3.3_SOT223, Package_TO_SOT_SMD:SOT-223-3_TabPin2, symbol Regulator_Linear:NCP1117-3.3_SOT223
- added U3: TP5400, Package_SO:SOIC-8_3.9x4.9mm_P1.27mm, symbol Interface_CAN_LIN:SN65HVD255D
- added U4: SIL2308, Package_TO_SOT_SMD:SOT-23-6, symbol Driver_FET:LTC4440ES6
- added U6: 74LVC1G14, Package_TO_SOT_SMD:SOT-23-5_HandSoldering, symbol 74xGxx:74LVC1G14
- added U7: 74LVC1G17, Package_TO_SOT_SMD:SOT-23-5_HandSoldering, symbol 74xGxx:74LVC1G17
- added U8: 74LVC1G175, Package_TO_SOT_SMD:TSOT-23-6_HandSoldering, symbol 74xGxx:74LVC1G175
- C1: value 10u -> 22uF; JLCPCB (none) -> C602037
- C10, C6, C7, C9: JLCPCB (none) -> C368809
- C11, C12, C13, C14, C15, C16, C17, C18, C2, C20, C21, C24, C79, C8: JLCPCB (none) -> C77020
- C19: JLCPCB (none) -> C17024
- C3, C4: JLCPCB (none) -> C86285
- C5: value 10u -> 100n; footprint Capacitor_SMD:C_0805_2012Metric -> Capacitor_SMD:C_0402_1005Metric; JLCPCB (none) -> C77020
- D1: JLCPCB (none) -> C2837790
- J1, J20, KP#1, KP*1, KP0, KP1, KP2, KP3, KP4, KP5, KP6, KP7, KP8, KP9, KPC1, KPDOWN1, KPSELECT1, KPUP1, LS2, M1: now left out of the parts list
- L1: JLCPCB (none) -> C42411119
- Q1: JLCPCB (none) -> C391423
- R1: value DNF -> 10k; JLCPCB (none) -> C60490
- R10: value 0 -> 220; JLCPCB (none) -> C137872
- R11, R12: value 90 -> 220; JLCPCB (none) -> C137872
- R13, R4, R5: value 140 -> 220; JLCPCB (none) -> C137872
- R14, R16, R19, R22: value 90 -> 1K; JLCPCB (none) -> C25543
- R15: value 90 -> 100k; JLCPCB (none) -> C25543
- R18: value 140 -> 100; JLCPCB (none) -> C25543
- R2: JLCPCB (none) -> C25543
- R20: value 90 -> 10k; JLCPCB (none) -> C25543
- R21: value 140 -> 200k; JLCPCB (none) -> C25543
- R3: JLCPCB (none) -> C852729
- R34, R35, R36, R38: JLCPCB (none) -> C60490
- R37: JLCPCB (none) -> C114758
- R39: JLCPCB (none) -> C60491
- R44, R45, R46, R47, R48, R49, R50, R51, R52, R53, R54, R55, R56, R57, R58, R59: JLCPCB (none) -> C137872
- R6: value 3k -> 220; JLCPCB (none) -> C137872
- R7, R8: JLCPCB (none) -> C25100
- R9: value DNF -> 220; JLCPCB (none) -> C137872
- SW1: JLCPCB (none) -> C128539
- TP1: footprint PiicoDev Real Time Clock RV3028:PinHeader_1x01_P2.54mm_Vertical -> TestPoint:TestPoint_THTPad_D1.5mm_Drill0.7mm
- U1: JLCPCB (none) -> C97521
- U5: JLCPCB (none) -> C42415655
- Y1: JLCPCB (none) -> C20625731
- Y2: JLCPCB (none) -> C3019759
Connections:
- net +3V3: now also C25.1, D2.2 (A), D3.2 (A), D4.2 (A), D5.2 (A), D6.2 (A), D7.2 (A), D8.2 (A), D9.2 (A), U2.2 (VO); no longer C5.1, J20.1 (Pin_1), R1.1, R6.1
- net GPIO0: now also J2.5 (Pin_5); no longer R9.1
- net GPIO1: now also J2.7 (Pin_7)
- net GPIO15: now also Q2.1 (B), Q5.1 (B), Q7.1 (B), Q9.1 (B)
- net GPIO34: now also J3.1 (Pin_1); no longer R12.1, R15.1, R20.1
- net QSPI_SS: now also R1.1, U1.1 (~{CS}); no longer R10.1
- net SWCLK: now also J2.2 (Pin_2)
- net SWD: now also J2.4 (Pin_4)
- net USB_D+: now also J5.3 (D+)
- net USB_D-: now also J5.2 (D-)
- net VBUS: now also J5.1 (VBUS), JP2.1 (A), U3.5 (VCC)
- net at R16.2: now also U4.1
- net at R12.2: now also D8.1 (K)
- net at R18.1: now also Q6.3 (D)
- net at R19.2: now also Q6.1 (G)
- net Off: now reaches R20.2
- net Off: now also R19.1
- net at R15.2: now also F1.1, U4.2
- net Btn: now reaches R21.1
- net Btn: now also R22.1, SW1.2, U5.36 (GPIO28), C34.1, D10.2 (A), U6.2
- net +5V: now reaches R22.2
- net +5V: now also C29.2, C30.2, C35.2, D12.1 (K), F1.2, J2.8 (Pin_8), JP2.2 (B), U3.1 (VOUT), U6.5 (VCC), U7.5 (VCC), U8.3 (D), U8.5 (VCC)
- net at R4.1: now also R5.1, Q2.3 (C)
- net at R11.2: now also D7.1 (K)
- net at R13.1: now also R6.1, Q9.3 (C)
- net at TP1.1: now also U3.2 (CHRG); no longer Y2.6 (VBACKUP)
- net at R14.2: now also U6.4, U8.1 (C)
- net ALARMB: no longer names the net of U5.54 (GPIO43_ADC3)
- net CLK: no longer names the net of Y2.1 (CLKOUT)
- removed net FLASH_SS: R1.2, R10.2, R9.2, U1.1 (~{CS})
- net GND renamed -BATT
- net -BATT: now also R20.1, C23.2, C25.2, C26.2, C27.2, C28.2, C29.1, C30.1, C31.2, C33.2, C34.2, C35.1, J2.1 (Pin_1), J2.3 (Pin_3), J2.6 (Pin_6), J3.2 (Pin_2), J5.5 (GND), J5.6 (Shield), Q2.2 (E), Q4.2 (S), Q5.2 (E), Q6.2 (S), Q7.2 (E), Q9.2 (E), R41.1, SW2.1, U2.1 (GND), U3.7 (GND), U4.5, U6.3 (GND), U7.3 (GND), U8.2 (GND)
- net GPIO22: no longer names the net of U5.22 (GPIO22)
- net GPIO23: no longer names the net of U5.23 (GPIO23)
- net GPIO24: no longer names the net of U5.25 (GPIO24)
- net GPIO25: no longer names the net of U5.26 (GPIO25)
- net GPIO26: no longer names the net of U5.27 (GPIO26)
- net GPIO27: no longer names the net of U5.28 (GPIO27)
- removed net GPIO28: R6.2, SW1.2, U5.36 (GPIO28)
- net GPIO29: no longer names the net of U5.37 (GPIO29)
- net GPIO3: no longer names the net of U5.80 (GPIO3)
- removed net GPIO30: R11.1, R14.1, R16.1, R19.1, R22.1, U5.38 (GPIO30)
- net GPIO31: no longer names the net of U5.39 (GPIO31)
- removed net GPIO32: R13.2, R18.2, R21.2, R4.2, R5.2, U5.40 (GPIO32)
- net GPIO35: no longer names the net of U5.44 (GPIO35)
- net GPIO40_ADC0: no longer names the net of U5.49 (GPIO40_ADC0)
- net GPIO41_ADC1: no longer names the net of U5.52 (GPIO41_ADC1)
- net SCL0: no longer names the net of U5.56 (GPIO45_ADC5)
- net SDA0: no longer names the net of U5.55 (GPIO44_ADC4)
- new net: Q7.3 (C), R11.1, R12.1
- new net: Q5.3 (C), R10.1, R9.1
- new net: D5.1 (K), R9.2
- new net: D2.1 (K), R4.2
- new net: D3.1 (K), R5.2
- new net: D4.1 (K), R6.2
- new net: Q4.1 (G), R14.1
- new net: R1.2, SW2.2
- new net: C23.1, U2.3 (VI), U4.4
- new net: C33.1, D10.1 (K), R18.2, R21.2, U7.2
- new net: U7.4, U8.6 (~{CLR})
- new net: D6.1 (K), R10.2
- new net: D9.1 (K), R13.2
- new net: TP2.1, U3.4 (STDBY)
- new net: D12.2 (A), L2.1, U3.8 (LX)
- new net: R41.2, U3.3 (PROG)
- new net: R15.1, U4.3, U4.6
- new net: C31.1, C5.1, TP3.1, Y2.6 (VBACKUP)
- new net +BATT: C26.1, C27.1, C28.1, J20.1 (Pin_1), L2.2, U3.6 (BAT)
- new net En: R16.1, U8.4 (Q)
- new net Push: Q4.3 (D)
- no-connect marks 4 -> 23
Other:
- note added: "Charging"
- note removed: "Clear jumper to remove I2C pullup"
- note removed: "JST Debug Connector"
- note removed: "Keypad"
- note removed: "Power"
- note removed: "UART Connector"
- moved on the sheet: C2, C24, C3, C4, C79, J20, KP#1, KP*1, KP0, KP1, KP2, KP3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
